File: stack-adapter/kicad/bobcat-rak-stack-adapter.kicad_pcb (KiCad board)
At the start: 2 copper layers, 31.3 x 60.3 mm, 13 parts, among them J1 PCIE-52P52H

Commit message: stack-adapter: GPS PPS to the processor (R47P fitted: RAK 19 -> finger 47 -> GPIO4_D0); docs: PPS/UART/qErr notes
Adapter: R47P 0R fitted, R45P (-> finger 45 / GPIO4_C7), R19, R23, R30-R33 DNP. Fingers 45/47 are their own
nets; the RAK's 45/47 come only from the SPI reroute of Bobcat 3/5. KiCad DRC 0 errors / 0 unconnected.
New docs/pps-uart-qerr.md: PPS path and core-3 capture, IO-voltage evidence, the GPS UART on RAK 31/33
(unmapped) with mapping method and fallback, and qErr (UBX-TIM-TP) sawtooth correction incl. the SX1303
latch and mandatory UBX checksum verification.

Co-Authored-By: Claude Opus 5.5 <noreply@anthropic.com>
Claude-Session: https://claude.ai/code/session_01Au7yLXRzrrweJwAkfxbhgS
Parts:
- added R45P: 0R DNP, tscircuit:resistor_res0402, F.Cu at (93.8, 112.3)
- added R47P: 0R, tscircuit:resistor_res0402, F.Cu at (91.6, 112.3)
Connections:
- CE2 pad 45: (no net) -> F45
- CE2 pad 47: (no net) -> F47
Routing:
- net F47: track 0.00 -> 33.3 mm, vias 0 -> 2
- net F45: track 0.00 -> 30.4 mm, vias 0 -> 2
- net V3V3: track 75.7 -> 96.3 mm, vias 6 -> 3
- net SPI_7_51: track 29.2 -> 43.6 mm
- net SPI_6_49: track 27.6 -> 41.5 mm, vias 1 -> 3
- net SPI_5_47: track 29.0 -> 40.1 mm, vias 2 -> 4
- net B31: track 25.8 -> 17.6 mm, vias 4 -> 2
- net B30: track 25.7 -> 18.8 mm, vias 3 -> 1
- net GND: track 147.0 -> 141.1 mm, vias 147 -> 148
- net B23: track 24.4 -> 19.0 mm
- net R19: track 13.2 -> 18.2 mm, vias 0 -> 2
- net B33: track 27.2 -> 22.3 mm, vias 4 -> 2
- net B32: track 20.5 -> 18.2 mm, vias 3 -> 1
- net R31: track 15.1 -> 12.9 mm
- net SPI_3_45: track 39.1 -> 41.1 mm
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Other:
- outline, holes or cut-outs redrawn
- board text added: "Mini CEM fig 2-7 top keep-out 3.20 (4.20 at key); tabs 0.30 from notch edge"
- board text added: "PPS: RAK19 → R47P → 47 → GPIO4_D0"
- board text added: "RAK socket front (pads/tabs): 4.20 mm (gap to the 2.55 mm fingers 1.65)"
- board text removed: "Mini Card top keep-out: 3.20 (4.20 at key)"
- board text removed: "RAK socket front (pads/tabs): 4.20 mm"

Commit message: stack-adapter: 2-up JLCPCB panel (78.7 x 60.4 mm, mouse-bites, fingers flush, rails + fiducials) with panel BOM/CPL
Gold-finger bevel needs >= 50 x 50 mm, so the 30 x 60.3 mm adapter ships 2-up. GND stitching kept >= 1 mm
from the outline (clears mouse-bites). KiCad DRC 0 errors / 0 unconnected; gerber_check passes incl. size.

Co-Authored-By: Claude Opus 5.5 <noreply@anthropic.com>
Claude-Session: https://claude.ai/code/session_01Au7yLXRzrrweJwAkfxbhgS
Routing:
- net GND: vias 148 -> 135
